File: OpenCAPI_Breakout.kicad_pcb (KiCad board)
At the start: 4 copper layers, 50 x 71 mm, 36 parts, among them J1 OpenCAPI_AAC_Host, J10 Rx3_N, J11 Rx4_P, J12 Rx4_N, J13 Rx5_P, J14 Rx5_N, J15 Rx6_P, J16 Rx6_N, J17 Rx7_P, J18 Rx7_N, J19 Tx0_P, J2 Conn_01x05, J20 Tx0_N, J21 Tx1_P, J22 Tx1_N, J23 Tx2_P, J24 Tx2_N, J25 Tx3_P, J26 Tx3_N, J27 Tx4_P, J28 Tx4_N, J29 Tx5_P, J3 Rx0_P, J30 Tx5_N, J31 Tx6_P, J32 Tx6_N, J33 Tx7_P, J34 Tx7_N, J35 CLK_P, J36 CLK_N, J4 Rx0_N, J5 Rx1_P, J6 Rx1_N, J7 Rx2_P, J8 Rx2_N, J9 Rx3_P

Commit message: Second Revision
Parts:
- J10: value Rx3_N -> Tx3_N
- J11: value Rx4_P -> Tx4_P
- J12: value Rx4_N -> Tx4_N
- J13: value Rx5_P -> Tx5_P
- J14: value Rx5_N -> Tx5_N
- J15: value Rx6_P -> Tx6_P
- J16: value Rx6_N -> Tx6_N
- J17: value Rx7_P -> Tx7_P
- J18: value Rx7_N -> Tx7_N
- J19: value Tx0_P -> Rx0_P
- J20: value Tx0_N -> Rx0_N
- J21: value Tx1_P -> Rx1_P
- J22: value Tx1_N -> Rx1_N
- J23: value Tx2_P -> Rx2_P
- J24: value Tx2_N -> Rx2_N
- J25: value Tx3_P -> Rx3_P
- J26: value Tx3_N -> Rx3_N
- J27: value Tx4_P -> Rx4_P
- J28: value Tx4_N -> Rx4_N
- J29: value Tx5_P -> Rx5_P
- J3: value Rx0_P -> Tx0_P
- J30: value Tx5_N -> Rx5_N
- J31: value Tx6_P -> Rx6_P
- J32: value Tx6_N -> Rx6_N
- J33: value Tx7_P -> Rx7_P
- J34: value Tx7_N -> Rx7_N
- J4: value Rx0_N -> Tx0_N
- J5: value Rx1_P -> Tx1_P
- J6: value Rx1_N -> Tx1_N
- J7: value Rx2_P -> Tx2_P
- J8: value Rx2_N -> Tx2_N
- J9: value Rx3_P -> Tx3_P
Routing:
- net GND: track 493.5 -> 498.4 mm, vias 249 -> 250
Other:
- board text added: "Channel X0Y_ Labels are for the Innova2 MNV303212A Rev.A2 Its Tx0, Tx3, and Tx4 _n,_p differential pairs are swapped"
- board text added: "OpenCAPI Breakout for AAC Add-In Cards"
- board text added: "OpenCAPI Connector Pin Mapping: Rx0p=B35, Rx0n=B36, Tx0p=A2, Tx0n=A3 Rx1p=B32, Rx1n=B33, Tx1p=B2, Tx1n=B3 Rx2p=A35, Rx2n=A36, Tx2p=A5, Tx2n=A6 Rx3p=B29, Rx3n=B30, Tx3p=B5, Tx3n=B6 Rx4p=B23, Rx4n=B24, Tx4p=B11, Tx4n=B12 Rx5p=A26, Rx5n=A27, Tx5p=A14, Tx5n=A15 Rx6p=B32, Rx6n=B33, Tx6p=B14, Tx6n=B15 Rx7p=A23, Rx7n=A24, Tx7p=A17, Tx7n=A18 REFCLK_P=A29, REFCLK_N=A30 SCL=B17, SDA=B18, RST=A21, PRE=A20 N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"
- board text added: "Ports are labelled with the Signal on them Tx connects to Add-In Card transmitter Rx connects to Add-In Card receiver"
- board text added: "X0Y16"
- board text added: "X0Y17"
- board text added: "X0Y18"
- board text added: "X0Y19"
- board text added: "X0Y20"
- board text added: "X0Y21"
- board text added: "X0Y22"
- board text added: "X0Y23"
- board text added: "_p _n"
- board text removed: "OpenCAPI HOST Pinout"
- board text removed: "OpenCAPI-Compatible SlimSAS 8x Breakout"
