File: OpenCAPI_Breakout.kicad_sch (KiCad schematic)
At the start: 36 parts, among them J1 OpenCAPI_AAC_Host, J10 Rx3_N, J11 Rx4_P, J12 Rx4_N, J13 Rx5_P, J14 Rx5_N, J15 Rx6_P, J16 Rx6_N, J17 Rx7_P, J18 Rx7_N, J19 Tx0_P, J2 Conn_01x05, J20 Tx0_N, J21 Tx1_P, J22 Tx1_N, J23 Tx2_P, J24 Tx2_N, J25 Tx3_P, J26 Tx3_N, J27 Tx4_P, J28 Tx4_N, J29 Tx5_P, J3 Rx0_P, J30 Tx5_N, J31 Tx6_P, J32 Tx6_N, J33 Tx7_P, J34 Tx7_N, J35 CLK_P, J36 CLK_N, J4 Rx0_N, J5 Rx1_P, J6 Rx1_N, J7 Rx2_P, J8 Rx2_N, J9 Rx3_P

Commit message: Second Revision
Parts:
- J10: value Rx3_N -> Tx3_N
- J11: value Rx4_P -> Tx4_P
- J12: value Rx4_N -> Tx4_N
- J13: value Rx5_P -> Tx5_P
- J14: value Rx5_N -> Tx5_N
- J15: value Rx6_P -> Tx6_P
- J16: value Rx6_N -> Tx6_N
- J17: value Rx7_P -> Tx7_P
- J18: value Rx7_N -> Tx7_N
- J19: value Tx0_P -> Rx0_P
- J20: value Tx0_N -> Rx0_N
- J21: value Tx1_P -> Rx1_P
- J22: value Tx1_N -> Rx1_N
- J23: value Tx2_P -> Rx2_P
- J24: value Tx2_N -> Rx2_N
- J25: value Tx3_P -> Rx3_P
- J26: value Tx3_N -> Rx3_N
- J27: value Tx4_P -> Rx4_P
- J28: value Tx4_N -> Rx4_N
- J29: value Tx5_P -> Rx5_P
- J3: value Rx0_P -> Tx0_P
- J30: value Tx5_N -> Rx5_N
- J31: value Tx6_P -> Rx6_P
- J32: value Tx6_N -> Rx6_N
- J33: value Tx7_P -> Rx7_P
- J34: value Tx7_N -> Rx7_N
- J4: value Rx0_N -> Tx0_N
- J5: value Rx1_P -> Tx1_P
- J6: value Rx1_N -> Tx1_N
- J7: value Rx2_P -> Tx2_P
- J8: value Rx2_N -> Tx2_N
- J9: value Rx3_P -> Tx3_P
Other:
- note added: "U.FL Connectors are Labelled according to the signal present on them. As this is an OpenCAPI AAC Carrier breakout, Host RX has TX signals present on it."
- moved on the sheet: J10, J11, J12, J13, J14, J15, J16, J17, J18, J19, J20, J21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
